Commit message: Add E1 SMPL-X retargeting support
Add E1 model marker updates, original model backups, SMPL-X assets via LFS, variable-DOF data conversion, and Viser playback/debug controls for mesh and mapped skeleton visualization.

File: src/holosoma_retargeting/holosoma_retargeting/models/e1/e1_23dof.urdf (robot description, URDF)
Before this commit: robot E1_111, 25 links, 24 joints
Links:
- added link l_foot_sphere_1_link, mass 0.001; visual sphere radius=0.005
- added link l_foot_sphere_2_link, mass 0.001; visual sphere radius=0.005
- added link l_foot_sphere_3_link, mass 0.001; visual sphere radius=0.005
- added link l_foot_sphere_4_link, mass 0.001; visual sphere radius=0.005
- added link l_foot_sphere_5_link, mass 0.001; visual sphere radius=0.005
- added link l_hand_sphere_link, mass 0.001; visual sphere radius=0.005
- added link l_leg_ankle_intermediate_1_link, mass 0.01; visual sphere radius=0.01
- added link r_foot_sphere_1_link, mass 0.001; visual sphere radius=0.005
- added link r_foot_sphere_2_link, mass 0.001; visual sphere radius=0.005
- added link r_foot_sphere_3_link, mass 0.001; visual sphere radius=0.005
- added link r_foot_sphere_4_link, mass 0.001; visual sphere radius=0.005
- added link r_foot_sphere_5_link, mass 0.001; visual sphere radius=0.005
- added link r_hand_sphere_link, mass 0.001; visual sphere radius=0.005
- added link r_leg_ankle_intermediate_1_link, mass 0.01; visual sphere radius=0.01
- link base_link: geometry collision mesh filename=meshes/base_link.STL; visual mesh filename=meshes/base_link.STL
- link l_arm_elbow_pitch_link: geometry collision mesh filename=meshes/l_arm_elbow_pitch_link.STL; visual mesh filename=meshes/l_arm_elbow_pitch_link.STL
- link l_arm_elbow_yaw_link: geometry collision mesh filename=meshes/l_arm_elbow_yaw_link.STL; visual mesh filename=meshes/l_arm_elbow_yaw_link.STL
- link l_arm_shoulder_pitch_link: geometry collision mesh filename=meshes/l_arm_shoulder_pitch_link.STL; visual mesh filename=meshes/l_arm_shoulder_pitch_link.STL
- link l_arm_shoulder_roll_link: geometry collision mesh filename=meshes/l_arm_shoulder_roll_link.STL; visual mesh filename=meshes/l_arm_shoulder_roll_link.STL
- link l_arm_shoulder_yaw_link: geometry collision mesh filename=meshes/l_arm_shoulder_yaw_link.STL; visual mesh filename=meshes/l_arm_shoulder_yaw_link.STL
- link l_leg_ankle_pitch_link: geometry collision mesh filename=meshes/l_leg_ankle_pitch_link.STL; visual mesh filename=meshes/l_leg_ankle_pitch_link.STL
- link l_leg_ankle_roll_link: geometry collision mesh filename=meshes/l_leg_ankle_roll_link.STL; visual mesh filename=meshes/l_leg_ankle_roll_link.STL
- link l_leg_hip_pitch_link: geometry collision mesh filename=meshes/l_leg_hip_pitch_link.STL; visual mesh filename=meshes/l_leg_hip_pitch_link.STL
- link l_leg_hip_roll_link: geometry collision mesh filename=meshes/l_leg_hip_roll_link.STL; visual mesh filename=meshes/l_leg_hip_roll_link.STL
- link l_leg_hip_yaw_link: geometry collision mesh filename=meshes/l_leg_hip_yaw_link.STL; visual mesh filename=meshes/l_leg_hip_yaw_link.STL
- link l_leg_knee_link: geometry collision mesh filename=meshes/l_leg_knee_link.STL; visual mesh filename=meshes/l_leg_knee_link.STL
- link r_arm_elbow_pitch_link: geometry collision mesh filename=meshes/r_arm_elbow_pitch_link.STL; visual mesh filename=meshes/r_arm_elbow_pitch_link.STL
- link r_arm_elbow_yaw_link: geometry collision mesh filename=meshes/r_arm_elbow_yaw_link.STL; visual mesh filename=meshes/r_arm_elbow_yaw_link.STL
- link r_arm_shoulder_pitch_link: geometry collision mesh filename=meshes/r_arm_shoulder_pitch_link.STL; visual mesh filename=meshes/r_arm_shoulder_pitch_link.STL
- link r_arm_shoulder_roll_link: geometry collision mesh filename=meshes/r_arm_shoulder_roll_link.STL; visual mesh filename=meshes/r_arm_shoulder_roll_link.STL
- link r_arm_shoulder_yaw_link: geometry collision mesh filename=meshes/r_arm_shoulder_yaw_link.STL; visual mesh filename=meshes/r_arm_shoulder_yaw_link.STL
- link r_leg_ankle_pitch_link: geometry collision mesh filename=meshes/r_leg_ankle_pitch_link.STL; visual mesh filename=meshes/r_leg_ankle_pitch_link.STL
- link r_leg_ankle_roll_link: geometry collision mesh filename=meshes/r_leg_ankle_roll_link.STL; visual mesh filename=meshes/r_leg_ankle_roll_link.STL
- link r_leg_hip_pitch_link: geometry collision mesh filename=meshes/r_leg_hip_pitch_link.STL; visual mesh filename=meshes/r_leg_hip_pitch_link.STL
- link r_leg_hip_roll_link: geometry collision mesh filename=meshes/r_leg_hip_roll_link.STL; visual mesh filename=meshes/r_leg_hip_roll_link.STL
- link r_leg_hip_yaw_link: geometry collision mesh filename=meshes/r_leg_hip_yaw_link.STL; visual mesh filename=meshes/r_leg_hip_yaw_link.STL
- link r_leg_knee_link: geometry collision mesh filename=meshes/r_leg_knee_link.STL; visual mesh filename=meshes/r_leg_knee_link.STL
- link waist_roll_link: geometry collision mesh filename=meshes/waist_roll_link.STL; visual mesh filename=meshes/waist_roll_link.STL
- link waist_yaw_link: geometry collision mesh filename=meshes/waist_yaw_link.STL; visual mesh filename=meshes/waist_yaw_link.STL
Joints:
- added joint l_foot_sphere_1_joint: type fixed, parent l_leg_ankle_roll_link, child l_foot_sphere_1_link, origin xyz=-0.055 0.025 -0.0495 rpy=0 0 0
- added joint l_foot_sphere_2_joint: type fixed, parent l_leg_ankle_roll_link, child l_foot_sphere_2_link, origin xyz=-0.055 -0.025 -0.0495 rpy=0 0 0
- added joint l_foot_sphere_3_joint: type fixed, parent l_leg_ankle_roll_link, child l_foot_sphere_3_link, origin xyz=0.115 0.025 -0.0495 rpy=0 0 0
- added joint l_foot_sphere_4_joint: type fixed, parent l_leg_ankle_roll_link, child l_foot_sphere_4_link, origin xyz=0.115 -0.025 -0.0495 rpy=0 0 0
- added joint l_foot_sphere_5_joint: type fixed, parent l_leg_ankle_roll_link, child l_foot_sphere_5_link, origin xyz=0.14 0 -0.0495 rpy=0 0 0
- added joint l_hand_sphere_joint: type fixed, parent l_arm_elbow_yaw_link, child l_hand_sphere_link, origin xyz=0 0 -0.11 rpy=0 0 0
- added joint l_leg_ankle_intermediate_1_joint: type fixed, parent l_leg_knee_link, child l_leg_ankle_intermediate_1_link, origin xyz=3.9185E-05 0.018243 -0.28 rpy=0 0 0
- added joint r_foot_sphere_1_joint: type fixed, parent r_leg_ankle_roll_link, child r_foot_sphere_1_link, origin xyz=-0.055 0.025 -0.0495 rpy=0 0 0
- added joint r_foot_sphere_2_joint: type fixed, parent r_leg_ankle_roll_link, child r_foot_sphere_2_link, origin xyz=-0.055 -0.025 -0.0495 rpy=0 0 0
- added joint r_foot_sphere_3_joint: type fixed, parent r_leg_ankle_roll_link, child r_foot_sphere_3_link, origin xyz=0.115 0.025 -0.0495 rpy=0 0 0
- added joint r_foot_sphere_4_joint: type fixed, parent r_leg_ankle_roll_link, child r_foot_sphere_4_link, origin xyz=0.115 -0.025 -0.0495 rpy=0 0 0
- added joint r_foot_sphere_5_joint: type fixed, parent r_leg_ankle_roll_link, child r_foot_sphere_5_link, origin xyz=0.14 0 -0.0495 rpy=0 0 0
- added joint r_hand_sphere_joint: type fixed, parent r_arm_elbow_yaw_link, child r_hand_sphere_link, origin xyz=0 0 -0.11 rpy=0 0 0
- added joint r_leg_ankle_intermediate_1_joint: type fixed, parent r_leg_knee_link, child r_leg_ankle_intermediate_1_link, origin xyz=3.9185E-05 -0.018242 -0.28 rpy=0 0 0

File: src/holosoma_retargeting/holosoma_retargeting/models/e1/e1_23dof_ori.urdf (robot description, URDF)
Before this commit: robot E1_111, 37 links, 36 joints
Links:
- removed link l_foot_sphere_1_link
- removed link l_foot_sphere_2_link
- removed link l_foot_sphere_3_link
- removed link l_foot_sphere_4_link
- removed link l_foot_sphere_5_link
- removed link l_hand_sphere_link
- removed link r_foot_sphere_1_link
- removed link r_foot_sphere_2_link
- removed link r_foot_sphere_3_link
- removed link r_foot_sphere_4_link
- removed link r_foot_sphere_5_link
- removed link r_hand_sphere_link
Joints:
- removed joint l_foot_sphere_1_joint
- removed joint l_foot_sphere_2_joint
- removed joint l_foot_sphere_3_joint
- removed joint l_foot_sphere_4_joint
- removed joint l_foot_sphere_5_joint
- removed joint l_hand_sphere_joint
- removed joint r_foot_sphere_1_joint
- removed joint r_foot_sphere_2_joint
- removed joint r_foot_sphere_3_joint
- removed joint r_foot_sphere_4_joint
- removed joint r_foot_sphere_5_joint
- removed joint r_hand_sphere_joint
