Commit message: Replace OMOMO global hulls with convex collision assets

File: src/holosoma_retargeting/holosoma_retargeting/models/clothesstand/clothesstand.urdf (robot description, URDF)
Before this commit: robot clothesstand, 1 links, 0 joints
Links:
- link clothesstand_link: geometry collision mesh filename=collision/clothesstand_collision_000.obj scale=1 1 1; collision mesh filename=collision/clothesstand_collision_001.obj scale=1 1 1

File: src/holosoma_retargeting/holosoma_retargeting/models/floorlamp/floorlamp.urdf (robot description, URDF)
Before this commit: robot floorlamp, 1 links, 0 joints
Links:
- link floorlamp_link: geometry collision mesh filename=collision/floorlamp_collision_000.obj scale=1 1 1; collision mesh filename=collision/floorlamp_collision_001.obj scale=1 1 1

File: src/holosoma_retargeting/holosoma_retargeting/models/largebox/largebox.urdf (robot description, URDF)
Before this commit: robot largebox, 1 links, 0 joints
Links:
- link largebox_link: geometry collision mesh filename=collision/largebox_collision_000.obj scale=1 1 1; collision mesh filename=collision/largebox_collision_001.obj scale=1 1 1

File: src/holosoma_retargeting/holosoma_retargeting/models/largetable/largetable.urdf (robot description, URDF)
Before this commit: robot largetable, 1 links, 0 joints
Links:
- link largetable_link: geometry collision mesh filename=collision/largetable_collision_000.obj scale=1 1 1; collision mesh filename=collision/largetable_collision_001.obj scale=1 1 1

File: src/holosoma_retargeting/holosoma_retargeting/models/monitor/monitor.urdf (robot description, URDF)
Before this commit: robot monitor, 1 links, 0 joints
Links:
- link monitor_link: geometry collision mesh filename=collision/monitor_collision_000.obj scale=1 1 1; collision mesh filename=collision/monitor_collision_001.obj scale=1 1 1

File: src/holosoma_retargeting/holosoma_retargeting/models/plasticbox/plasticbox.urdf (robot description, URDF)
Before this commit: robot plasticbox, 1 links, 0 joints
Links:
- link plasticbox_link: geometry collision mesh filename=collision/plasticbox_collision_000.obj scale=1 1 1; collision mesh filename=collision/plasticbox_collision_001.obj scale=1 1 1

File: src/holosoma_retargeting/holosoma_retargeting/models/smallbox/smallbox.urdf (robot description, URDF)
Before this commit: robot smallbox, 1 links, 0 joints
Links:
- link smallbox_link: geometry collision mesh filename=collision/smallbox_collision_000.obj scale=1 1 1; collision mesh filename=collision/smallbox_collision_001.obj scale=1 1 1

File: src/holosoma_retargeting/holosoma_retargeting/models/smalltable/smalltable.urdf (robot description, URDF)
Before this commit: robot smalltable, 1 links, 0 joints
Links:
- link smalltable_link: geometry collision mesh filename=collision/smalltable_collision_000.obj scale=1 1 1; collision mesh filename=collision/smalltable_collision_001.obj scale=1 1 1

File: src/holosoma_retargeting/holosoma_retargeting/models/suitcase/suitcase.urdf (robot description, URDF)
Before this commit: robot suitcase, 1 links, 0 joints
Links:
- link suitcase_link: geometry collision mesh filename=collision/suitcase_collision_000.obj scale=1 1 1; collision mesh filename=collision/suitcase_collision_001.obj scale=1 1 1

File: src/holosoma_retargeting/holosoma_retargeting/models/trashcan/trashcan.urdf (robot description, URDF)
Before this commit: robot trashcan, 1 links, 0 joints
Links:
- link trashcan_link: geometry collision mesh filename=collision/trashcan_collision_000.obj scale=1 1 1; collision mesh filename=collision/trashcan_collision_001.obj scale=1 1 1

File: src/holosoma_retargeting/holosoma_retargeting/models/tripod/tripod.urdf (robot description, URDF)
Before this commit: robot tripod, 1 links, 0 joints
Links:
- link tripod_link: geometry collision mesh filename=collision/tripod_collision_000.obj scale=1 1 1; collision mesh filename=collision/tripod_collision_001.obj scale=1 1 1

File: src/holosoma_retargeting/holosoma_retargeting/models/whitechair/whitechair.urdf (robot description, URDF)
Before this commit: robot whitechair, 1 links, 0 joints
Links:
- link whitechair_link: geometry collision mesh filename=collision/whitechair_collision_000.obj scale=1 1 1; collision mesh filename=collision/whitechair_collision_001.obj scale=1 1 1

File: src/holosoma_retargeting/holosoma_retargeting/models/woodchair/woodchair.urdf (robot description, URDF)
Before this commit: robot woodchair, 1 links, 0 joints
Links:
- link woodchair_link: geometry collision mesh filename=collision/woodchair_collision_000.obj scale=1 1 1; collision mesh filename=collision/woodchair_collision_001.obj scale=1 1 1
